File: hardware/alarm_system_hardware/alarm_system_hardware.kicad_sch (KiCad schematic)
At the start: 113 parts, among them IC1 PCA9955BTW, J1 Micro_SD_Card_Det2, J2 USB_C_Receptacle_USB2.0_14P, J3 Conn_01x04_Socket, J4 Conn_01x02_Socket, J5 Conn_01x02_Socket, J6 Conn_01x02_Socket, Q1 NMOS, Q2 NMOS, Q3 NMOS, Q4 NMOS, Q5 NMOS, Q6 NMOS, SW1 SW_SPST, SW2 SW_SPST, SW3 SW_SPST, SW4 SW_Reed_Opener, SW7 SW_Push, SW8 SW_Push, U10 TMUX1204DQAR, U2 ESP32-S3-WROOM-1-N8R8, U3 MAX98357A, U4 BQ25616JRTWR, U6 TUSB321AIRWBR, U7 USBLC6-4SC6

Commit message: Add footprints for remaining parts
Parts:
- removed D1, D2, D3: LTST-C235KGKRKT, LED_SMD:LED_LiteOn_LTST-C235KGKRKT, symbol LED:LTST-C235KGKRKT
- removed D10: D_Schottky, symbol Device:D_Schottky
- removed Q1, Q2, Q3, Q4, Q5, Q6: NMOS, symbol Simulation_SPICE:NMOS
- removed R12, R13, R14, R15, R16, R17: 330, symbol Device:R_US
- added C21: 22uF, Capacitor_SMD:C_0805_2012Metric_Pad1.18x1.45mm_HandSolder, symbol Device:C_Small
- added C22: 0.1uF, Capacitor_SMD:C_0805_2012Metric_Pad1.18x1.45mm_HandSolder, symbol Device:C_Small
- added C7: 10uF, Capacitor_SMD:C_0805_2012Metric_Pad1.18x1.45mm_HandSolder, symbol Device:C_Small
- added L2: 0.47uH, alarm_system:IND_IHLP-2020CZ-L, symbol Device:L
- added R39: 0, Resistor_SMD:R_0805_2012Metric_Pad1.20x1.40mm_HandSolder, symbol Device:R_US
- added R40: NC, Resistor_SMD:R_0805_2012Metric_Pad1.20x1.40mm_HandSolder, symbol Device:R_US
- added R41: 511k, Resistor_SMD:R_0805_2012Metric_Pad1.20x1.40mm_HandSolder, symbol Device:R_US
- added R42: 91k, Resistor_SMD:R_0805_2012Metric_Pad1.20x1.40mm_HandSolder, symbol Device:R_US
- added U1: TPS63802DLAR, DLA0010A, symbol regulator_3v3:TPS63802DLAR
- C1, C10, C11, C12, C13, C14, C15, C16, C17, C18, C19, C2, C20, C3, C4, C5, C6, C8, C9: footprint (none) -> Capacitor_SMD:C_0805_2012Metric_Pad1.18x1.45mm_HandSolder
- D11, D15, D4, D5, D6, D7, D8: footprint (none) -> LED_SMD:LED_0805_2012Metric
- D9: footprint (none) -> Diode_SMD:D_SOD-323_HandSoldering
- F1: footprint (none) -> Fuse:Fuse_0805_2012Metric
- FB1: footprint (none) -> Resistor_SMD:R_1206_3216Metric_Pad1.30x1.75mm_HandSolder
- J1: footprint (none) -> alarm_system:CUI_MSD-11-A
- J2: value USB_C_Receptacle_USB2.0_14P -> USB_C_Receptacle_USB2.0_16P; footprint (none) -> alarm_system:SAMESKY_UJ20-C-H-G-SMT-1-P16-TR
- J3: footprint (none) -> Connector_PinHeader_2.54mm:PinHeader_1x04_P2.54mm_Vertical
- J4, J5, J6, SW4: footprint (none) -> TerminalBlock_Phoenix:TerminalBlock_Phoenix_PT-1,5-2-5.0-H_1x02_P5.00mm_Horizontal
- L1: footprint (none) -> alarm_system:IND_VLS5045EX-1R0N
- R1, R10, R11, R18, R19, R2, R20, R21, R22, R23, R24, R26, R29, R3, R30, R32, R34, R35, R36, R4, R44, R45, R46, R47, R48, R49, R5, R50, R6, R7, R8, R9: footprint (none) -> Resistor_SMD:R_0805_2012Metric_Pad1.20x1.40mm_HandSolder
- R25: value 900k -> 909k; footprint (none) -> Resistor_SMD:R_0805_2012Metric_Pad1.20x1.40mm_HandSolder
- R27, R28: value 300k -> 200k; footprint (none) -> Resistor_SMD:R_0805_2012Metric_Pad1.20x1.40mm_HandSolder
- R31, R33: value 10k -> 200; footprint (none) -> Resistor_SMD:R_0805_2012Metric_Pad1.20x1.40mm_HandSolder
- R37: value 5.3k -> 5.36k; footprint (none) -> Resistor_SMD:R_0805_2012Metric_Pad1.20x1.40mm_HandSolder
- R38: value 31.14k -> 31.6k; footprint (none) -> Resistor_SMD:R_0805_2012Metric_Pad1.20x1.40mm_HandSolder
- SW1, SW2, SW3: footprint (none) -> Button_Switch_THT:Push_E-Switch_KS01Q01
- SW7, SW8: value SW_Push -> SW_Tactile; footprint (none) -> Button_Switch_SMD:SW_SPST_CK_RS282G05A3
Connections:
- net UBSC_VBUS_PRE_DIODE is gone; now on net UBSC_VBUS: C11.1, C16.1, C17.1, FB1.2, R25.1, R49.1, R50.1, U10.5 (EN), U10.6 (VDD), U6.12 (VDD)
- net +3V3: now also C22.1
- net GND: now also C21.2, C22.2, C7.2, R39.2, U1.8 (GND)
- net GNDA: now also R42.2, U1.3 (AGND)
- net CHARGER_POWER: now reaches C12.1, L1.2, U4.15 (SYS), U4.16 (SYS)
- net CHARGER_POWER: now also C7.1, R40.1, U1.1 (EN), U1.10 (VIN)
- new net: C21.1, R41.1, U1.6 (VOUT)
- new net: R39.1, R40.2, U1.2 (MODE)
- new net: R41.2, R42.1, U1.4 (FB)
- new net: L2.2, U1.7 (L2)
- new net: L2.1, U1.9 (L1)
- no-connect marks 22 -> 23
Other:
- note added: "SYS Output Votlage Conclusion: - From battery conditions, downstream regulators should bet speced from about 2.18V to 4.7V (V_SYS_OVP is 4.7V caused by potential transients and voltage spikes)"
- note added: "TODO: - Consider adding PMOS on battery connector to prevent reverse polarity connection - CAUTION resistor on NTC connector was changed form 5.3k (datasheet recommendation) to 5.36k, verify this value works before being reliant on this; The 3.14k was also changed to 31.6k."
- note removed: "Button LED Indicators (ALT APPROACH)"
- note removed: "Host Protection"
- note removed: "TODO: - Make ILIM dynamic to handle 500mA, 1.5A, and 3A for various usb-c charger"
- note removed: "TODO: Connect All IO's to MCU"
- note removed: "TODO: Connect to MCU"
- moved on the sheet: C10, C12, C13, C14, C15, C16, C17, C18, C19, C20, C3, C4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
