File: hardware/alarm_system_hardware/alarm_system_hardware.kicad_sch (KiCad schematic)
At the start: 106 parts, among them IC1 PCA9955BTW, J1 Micro_SD_Card_Det2, J2 USB_C_Receptacle_USB2.0_16P, J3 Conn_01x04_Socket, J4 Conn_01x02_Socket, J5 Conn_01x02_Socket, J6 Conn_01x02_Socket, SW1 SW_SPST, SW2 SW_SPST, SW3 SW_SPST, SW4 SW_Reed_Opener, SW7 SW_Tactile, SW8 SW_Tactile, U1 TPS63802DLAR, U10 TMUX1204DQAR, U2 ESP32-S3-WROOM-1-N8R8, U3 MAX98357A, U4 BQ25616JRTWR, U6 TUSB321AIRWBR, U7 USBLC6-4SC6

Commit message: Completed V0.01 PCB and production files
Parts:
- removed D12, D13, D14: LTST-C235KGKRKT, LED_SMD:LED_LiteOn_LTST-C235KGKRKT, symbol LED:LTST-C235KGKRKT
- removed J1: Micro_SD_Card_Det2, alarm_system:CUI_MSD-11-A, symbol Connector:Micro_SD_Card_Det2
- removed J3: Conn_01x04_Socket, Connector_PinHeader_2.54mm:PinHeader_1x04_P2.54mm_Vertical, symbol Connector:Conn_01x04_Socket
- removed J5, J6: Conn_01x02_Socket, TerminalBlock_Phoenix:TerminalBlock_Phoenix_PT-1,5-2-5.0-H_1x02_P5.00mm_Horizontal, symbol Connector:Conn_01x02_Socket
- removed U7: USBLC6-4SC6, Package_TO_SOT_SMD:SOT-23-6, symbol Power_Protection:USBLC6-4SC6
- added BZ1: Buzzer, alarm_system:PS1440P02BT_TDK, symbol Device:Buzzer
- added C23: 1uF, Capacitor_SMD:C_0805_2012Metric_Pad1.18x1.45mm_HandSolder, symbol Device:C_Small
- added C24: 10uF, Capacitor_SMD:C_0805_2012Metric_Pad1.18x1.45mm_HandSolder, symbol Device:C_Small
- added D1, D2, D3: GREEN LED, LED_SMD:LED_0805_2012Metric, symbol Device:LED
- added D10, D12, D13: RED LED, LED_SMD:LED_0805_2012Metric, symbol Device:LED
- added J1: Conn_02x04_Odd_Even, Connector_PinHeader_2.54mm:PinHeader_2x04_P2.54mm_Vertical, symbol Connector_Generic:Conn_02x04_Odd_Even
- added J5: MSD-11-A, alarm_system:CUI_MSD-11-A, symbol micro_sd:MSD-11-A
- added J7: Conn_01x03_Socket, TerminalBlock_Phoenix:TerminalBlock_Phoenix_PT-1,5-3-3.5-H_1x03_P3.50mm_Horizontal, symbol Connector:Conn_01x03_Socket
- added Q1: AO3400A, Package_TO_SOT_SMD:SOT-23-3, symbol Simulation_SPICE:NMOS
- added R12: 8.25k, Resistor_SMD:R_0805_2012Metric_Pad1.20x1.40mm_HandSolder, symbol Device:R_US
- added R13, R53: 330, Resistor_SMD:R_0805_2012Metric_Pad1.20x1.40mm_HandSolder, symbol Device:R_US
- added R14, R15, R54: 100k, Resistor_SMD:R_0805_2012Metric_Pad1.20x1.40mm_HandSolder, symbol Device:R_US
- added R16, R17, R43, R51, R52: 0, Resistor_SMD:R_0805_2012Metric_Pad1.20x1.40mm_HandSolder, symbol Device:R_US
- added SW5: SW_SPST, Button_Switch_SMD:SW_SPST_CK_RS282G05A3, symbol Switch:SW_SPST
- added TP10, TP7, TP8, TP9: TestPoint, TestPoint:TestPoint_Pad_D1.0mm, symbol Connector:TestPoint
- added U5: PESD4USB5BTBS-QX, Package_DFN_QFN:Diodes_UDFN-10_1.0x2.5mm_P0.5mm, symbol Power_Protection:D3V3XA4B10LP
- J4: footprint TerminalBlock_Phoenix:TerminalBlock_Phoenix_PT-1,5-2-5.0-H_1x02_P5.00mm_Horizontal -> alarm_system:CONN_S2B-PH-K-S_JST
- R22: value 0 -> 1k; now not fitted
- SW1, SW2, SW3: footprint Button_Switch_THT:Push_E-Switch_KS01Q01 -> Button_Switch_SMD:SW_SPST_CK_RS282G05A3
- TP1, TP2, TP3, TP4, TP5, TP6: footprint (none) -> TestPoint:TestPoint_Pad_D1.0mm
Connections:
- net GNDA is gone; now on net COVER_GND: C14.2, R30.2, R32.2, R35.2, R36.2, R38.2, R42.2, U1.3 (AGND)
- net +3V3: now also R22.1, BZ1.1 (+), D1.2 (A), D10.2 (A), D12.2 (A), D13.2 (A), D2.2 (A), D3.2 (A), J1.2 (Pin_2), R12.1, R16.2, R17.2, R43.2, R51.2, R52.2; no longer C1.1, C18.1, C19.1, C2.1, C22.1, C6.1, C9.1, IC1.28 (VDD), R18.1, R24.1, U2.2 (3V3), U3.7 (VDD), U3.8 (VDD)
- net ARM_SWITCH: now also R8.2, U2.19 (IO11); no longer R7.2, U2.33 (IO40)
- net AUDIO_ON_OFF_SWITCH: now also U2.18 (IO10); no longer U2.35 (IO42)
- net DAC_!SD_BOOT: now also U2.20 (IO12); no longer U2.24 (IO47)
- net ESP_BCLK: now also U2.24 (IO47); no longer U2.19 (IO11)
- net ESP_DIN: now also U2.23 (IO21); no longer U2.18 (IO10)
- net ESP_LRCLK: now also U2.25 (IO48); no longer U2.20 (IO12)
- net ESP_RXD0: now also J1.4 (Pin_4)
- net ESP_TXD0: now also J1.6 (Pin_6)
- net LED_!OE: now also U2.11 (IO18); no longer U2.31 (IO38)
- net NOTIFICATIONS_SWITCH: now also R7.2, U2.17 (IO9); no longer R8.2, U2.34 (IO41)
- net REED_INPUT: now also U2.7 (IO7); no longer U2.25 (IO48)
- net SCL: now also U2.9 (IO16); no longer U2.38 (IO2)
- net SDA: now also U2.8 (IO15); no longer U2.39 (IO1)
- net SDCARD_CD/CS: now also U2.6 (IO6), J5.P2 (CD/DAT3); no longer U2.4 (IO4)
- net SDCARD_CLK: now also U2.38 (IO2), J5.P5 (CLK); no longer U2.6 (IO6)
- net SDCARD_MISO: now also U2.31 (IO38), J5.P7 (DAT0); no longer U2.7 (IO7)
- net SDCARD_MOSI: now also U2.39 (IO1), J5.P3 (CMD); no longer U2.5 (IO5)
- net USBC_CC1: now also U5.5, U5.6 (NC)
- net USBC_CC2: now also U5.4, U5.7 (NC)
- net USB_D+: now also U5.2, U5.9 (NC)
- net USB_D-: now also U5.1, U5.10 (NC)
- net at IC1.17 (LED10): now also D10.1 (K)
- net at IC1.18 (LED11): now also D1.1 (K)
- net at IC1.20 (LED12): now also D12.1 (K)
- net at IC1.21 (LED13): now also D2.1 (K)
- net at IC1.22 (LED14): now also D13.1 (K)
- net at IC1.23 (LED15): now also D3.1 (K)
- net TS: now reaches R37.2, R38.1, U4.11 (TS)
- net TS: now also J7.1 (Pin_1)
- net at F1.1, U4.13 (BAT), U4.14 (BAT): now also C24.1
- net at C21.1, R41.1, U1.6 (VOUT): now also R16.1
- net BUZZER_GPIO: now reaches U2.10 (IO17)
- net BUZZER_GPIO: now also R53.2, R54.1
- net BATTERY_LIFE_SWITCH: now reaches U2.15 (IO3)
- net BATTERY_LIFE_SWITCH: now also R13.2
- net JTAG_MTMS: now reaches U2.32 (IO39)
- net JTAG_MTMS: now also J1.7 (Pin_7)
- net USBC_VBUS: now reaches D9.1 (K), FB1.1, J2.A4 (VBUS), J2.A9 (VBUS), J2.B4 (VBUS), J2.B9 (VBUS)
- net COVER_GND: now reaches J2.S1 (SHIELD)
- net COVER_GND: now also C1.2, C10.2, C11.2, C12.2, C15.2, C16.2, C17.2, C18.2, C19.2, C2.2, C20.2, C21.2, C22.2, C3.2, C4.2, C5.2, C6.2, C7.2, C8.2, C9.2, D9.2 (A), IC1.10 (VSS_1), IC1.19 (VSS_2), IC1.2 (AD0), IC1.24 (VSS_3), IC1.29 (VSS_4), IC1.3 (AD1), IC1.4 (AD2), J2.A1 (GND), J2.A12 (GND), J2.B1 (GND), J2.B12 (GND), R20.1, R29.2, R39.2, R44.2, R45.1, R46.1, R47.2, R48.2, SW1.1 (A), SW2.1 (A), SW3.1 (A), SW4.2, SW7.2, SW8.2, U1.8 (GND), U10.3 (GND), U2.1 (GND), U2.40 (GND), U2.41 (GND), U3.11 (GND), U3.15 (GND), U3.17 (PAD), U3.3 (GND), U4.17 (GND), U4.18 (GND), U4.25 (GND), U6.10 (GND), U6.4 (PORT), C23.2, C24.2, J1.8 (Pin_8), J5.G1 (COVER_GND), J5.G2 (COVER_GND), J5.P6 (VSS), J7.3 (Pin_3), Q1.3 (S), R15.2, R54.2, SW5.1 (A), U5.3 (VSS), U5.8 (VSS); no longer R22.1
- net at U6.11 (DIR): now also TP10.1
- net at U6.3 (CURRENT_MODE): now also TP9.1
- net at U6.6 (~{VCONN_FAULT}): now also TP7.1
- net at U6.9 (ID): now also TP8.1
- net V_BAT: now reaches F1.2
- net V_BAT: now also J7.2 (Pin_2), R14.1
- net ESP_IO0 renamed ESP_BOOT
- removed net GND: C1.2, C10.2, C11.2, C12.2, C15.2, C16.2, C17.2, C18.2, C19.2, C2.2, C20.2, C21.2, C22.2, C3.2, C4.2, C5.2, C6.2, C7.2, C8.2, C9.2, D9.2 (A), IC1.10 (VSS_1), IC1.19 (VSS_2), IC1.2 (AD0), IC1.24 (VSS_3), IC1.29 (VSS_4), IC1.3 (AD1), IC1.4 (AD2), J2.A1 (GND), J2.A12 (GND), J2.B1 (GND), J2.B12 (GND), R20.1, R22.2, R29.2, R39.2, R44.2, R45.1, R46.1, R47.2, R48.2, SW1.1 (A), SW2.1 (A), SW3.1 (A), SW4.2, SW7.2, SW8.2, U1.8 (GND), U10.3 (GND), U2.1 (GND), U2.40 (GND), U2.41 (GND), U3.11 (GND), U3.15 (GND), U3.17 (PAD), U3.3 (GND), U4.17 (GND), U4.18 (GND), U4.25 (GND), U6.10 (GND), U6.4 (PORT)
- removed net SDCARD_GPIOX: R1.2, R2.2, U2.12 (IO8), U2.17 (IO9)
- removed net TODO_CRYSTAL: U2.8 (IO15), U2.9 (IO16)
- new net: Q1.2 (G), R53.1
- new net: C1.1, C2.1, J5.P4 (VDD), R52.1
- new net: C22.1, IC1.28 (VDD), R17.1, R18.1
- new net: C23.1, R12.2, R13.1, SW5.2 (B)
- new net: C18.1, C19.1, R24.1, R43.1, U2.2 (3V3)
- new net: C6.1, C9.1, R51.1, U3.7 (VDD), U3.8 (VDD)
- new net: BZ1.2 (-), Q1.1 (D), R22.2
- new net JTAG_MTCK: J1.1 (Pin_1), U2.35 (IO42)
- new net JTAG_MTDI: J1.5 (Pin_5), U2.33 (IO40)
- new net JTAG_MTDO: J1.3 (Pin_3), U2.34 (IO41)
- new net SDCARD_CD: J5.CD, R2.2, U2.4 (IO4)
- new net SDCARD_WP: J5.WP, R1.2, U2.5 (IO5)
- new net V_BAT_ADC: R14.2, R15.1, U2.12 (IO8)
- no-connect marks 23 -> 16
Other:
- note added: "For power measurements"
- note added: "JTAG Interface"
- note added: "LED Driver"
- note added: "Micro SD Card Interface"
- note added: "Mirco SD Card"
- note added: "NOTE: - This symbols internal electrical representation is innacturate to the actual part number. - The signals are routed through the no connects hence the labels attached there."
- note added: "NOTE: WP and CD connected to ground when micro sd card is inserted, otherwise they are floating. These can be read and OR'd together for added reduncancy."
- note added: "Passive Buzzer"
- note added: "Simple Battery Life Measurement"
- note added: "User Input"
- note removed: "LED_Driver"
- note removed: "NOTE: Both DET_A and Both DET_B will connect to ground under normal operating conditions when an SD card is inserted. These can be read and OR'd together for added reduncancy."
- note removed: "SD Card Interface"
- note removed: "SD_Card"
- note removed: "TODO: - Connect DET_A and DET_B to MCU - Connect SHIELD to ground?"
- note removed: "User Inputs"
- moved on the sheet: C1, C2, C3, C4, C5, D9, F1, R1, R10, R11, R2, R21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

Commit message: PCBA export file and related hardware changes
Parts:
- BZ1: Manufacturer_Name (none) -> TDK; Manufacturer_Part_Number (none) -> PS1440P02BT
- C1, C16, C17, C18, C22, C6, C8: Manufacturer_Name (none) -> YAGEO; Manufacturer_Part_Number (none) -> CC0805KRX7R9BB104
- C10, C2, C23, C3, C4, C5: Manufacturer_Name (none) -> Murata Electronics; Manufacturer_Part_Number (none) -> GRM21BR71C105KA01L
- C11, C12, C15, C24, C7, C9: Manufacturer_Name (none) -> Murata Electronics; Manufacturer_Part_Number (none) -> GRM21BR71A106KA73L
- C13, C14: Manufacturer_Name (none) -> Samsung Electro-Mechanics; Manufacturer_Part_Number (none) -> CL21B473KBCNNNC
- C19, C21: Manufacturer_Name (none) -> Murata Electronics; Manufacturer_Part_Number (none) -> GRM21BZ71A226ME15L
- C20: Manufacturer_Name (none) -> Murata Electronics; Manufacturer_Part_Number (none) -> GRM21BR71C105KA01L; now not fitted; now left out of the parts list
- D1, D2, D3: Manufacturer_Name (none) -> Lite-On Inc.; Manufacturer_Part_Number (none) -> LTST-C171KGKT
- D10, D12, D13: Manufacturer_Name (none) -> Lite-On Inc.; Manufacturer_Part_Number (none) -> LTST-C171KRKT
- D11, D15, D4, D5, D6, D7, D8: value LED -> GREEN LED; Manufacturer_Name (none) -> Lite-On Inc.; Manufacturer_Part_Number (none) -> LTST-C171KGKT
- D9: Manufacturer_Name (none) -> Texas Instruments; Manufacturer_Part_Number (none) -> TSD05DYFR
- F1: Manufacturer_Name (none) -> Vishay; Manufacturer_Part_Number (none) -> MFU0805FF03000P500
- FB1: Manufacturer_Name (none) -> Pulse Electronics; Manufacturer_Part_Number (none) -> BBUP00321611121Y00
- IC1: value PCA9955BTW -> PCA9955BTWJ; Manufacturer_Name NXP -> NXP USA Inc.; Manufacturer_Part_Number PCA9955BTW -> PCA9955BTWJ
- J1, R40: now not fitted; now left out of the parts list
- J2: Manufacturer_Name (none) -> Same Sky (Formerly CUI Devices); Manufacturer_Part_Number (none) -> UJ20-C-H-G-SMT-1-P16-TR
- J4: Manufacturer_Name (none) -> JST Sales America Inc.; Manufacturer_Part_Number (none) -> S2B-PH-K-S
- J5: Manufacturer_Name (none) -> Same Sky (Formerly CUI Devices); Manufacturer_Part_Number (none) -> MSD-11-A
- J7: footprint TerminalBlock_Phoenix:TerminalBlock_Phoenix_PT-1,5-3-3.5-H_1x03_P3.50mm_Horizontal -> TerminalBlock_Phoenix:TerminalBlock_Phoenix_PT-1,5-3-5.0-H_1x03_P5.00mm_Horizontal; Manufacturer_Name (none) -> Phoenix Contact; Manufacturer_Part_Number (none) -> 1935174
- L1: Manufacturer_Name (none) -> TDK; Manufacturer_Part_Number (none) -> VLS5045EX-1R0N
- L2: LCSC Part # (none) -> C5298158; Manufacturer_Name (none) -> Vishay Dale; Manufacturer_Part_Number (none) -> IHLP2020CZERR47M11
- Q1: Manufacturer_Name (none) -> Alpha & Omega Semiconductor Inc.; Manufacturer_Part_Number (none) -> AO3400A
- R1, R18, R19, R2, R24, R3, R30: Manufacturer_Name (none) -> Stackpole Electronics Inc; Manufacturer_Part_Number (none) -> RMCF0805FT10K0
- R10, R13, R53, R7, R8, R9: Manufacturer_Name (none) -> YAGEO; Manufacturer_Part_Number (none) -> RC0805JR-07330RL
- R11: Manufacturer_Name (none) -> YAGEO; Manufacturer_Part_Number (none) -> RC0805FR-0747KL
- R12, R4, R5, R6: Manufacturer_Name (none) -> YAGEO; Manufacturer_Part_Number (none) -> RT0805BRD078K25L
- R14, R15, R29, R32, R54: Manufacturer_Name (none) -> YAGEO; Manufacturer_Part_Number (none) -> RC0805FR-07100KL
- R16, R17, R35, R39, R43, R51, R52: Manufacturer_Name (none) -> YAGEO; Manufacturer_Part_Number (none) -> RC0805JR-070RL
- R20: Manufacturer_Name (none) -> YAGEO; Manufacturer_Part_Number (none) -> RC0805FR-072KL
- R21, R23: Manufacturer_Name (none) -> YAGEO; Manufacturer_Part_Number (none) -> RC0805FR-074K7L
- R22, TP1, TP10, TP2, TP3, TP4, TP5, TP6, TP7, TP8, TP9: now left out of the parts list
- R25: Manufacturer_Name (none) -> YAGEO; Manufacturer_Part_Number (none) -> RC0805FR-07909KL
- R26, R34: Manufacturer_Name (none) -> Stackpole Electronics Inc; Manufacturer_Part_Number (none) -> RMCF0805FT10K0; now not fitted; now left out of the parts list
- R27, R28: value 200k -> 100k; Manufacturer_Name (none) -> YAGEO; Manufacturer_Part_Number (none) -> RC0805FR-07100KL
- R31, R33, R45: Manufacturer_Name (none) -> YAGEO; Manufacturer_Part_Number (none) -> RC0805FR-07200RL
- R36: Manufacturer_Name (none) -> YAGEO; Manufacturer_Part_Number (none) -> RC0805FR-07432RL
- R37: Manufacturer_Name (none) -> Vishay Dale; Manufacturer_Part_Number (none) -> CRCW08055K36FKEA
- R38: Manufacturer_Name (none) -> YAGEO; Manufacturer_Part_Number (none) -> RC0805FR-0731K6L
- R41: Manufacturer_Name (none) -> YAGEO; Manufacturer_Part_Number (none) -> RC0805FR-07511KL
- R42: Manufacturer_Name (none) -> YAGEO; Manufacturer_Part_Number (none) -> RC0805FR-0791KL
- R44: Manufacturer_Name (none) -> YAGEO; Manufacturer_Part_Number (none) -> RC0805FR-071K05L
- R46: Manufacturer_Name (none) -> YAGEO; Manufacturer_Part_Number (none) -> RC0805FR-07499RL
- R47, R48: Manufacturer_Name (none) -> YAGEO; Manufacturer_Part_Number (none) -> RC0805FR-0710ML
- R49, R50: Manufacturer_Name (none) -> YAGEO; Manufacturer_Part_Number (none) -> RC0805FR-07200KL
- SW1, SW2, SW3, SW5: Manufacturer_Name (none) -> C&K; Manufacturer_Part_Number (none) -> PTS636SK25FSMTR LFS
- SW4: Manufacturer_Name (none) -> Phoenix Contact; Manufacturer_Part_Number (none) -> 1935161
- SW7, SW8: value SW_Tactile -> SW_SPST; Manufacturer_Name (none) -> C&K; Manufacturer_Part_Number (none) -> PTS636SK25FSMTR LFS
- U1: Manufacturer_Name (none) -> Texas Instruments; Manufacturer_Part_Number (none) -> TPS63802DLAR
- U10: Manufacturer_Name (none) -> Texas Instruments; Manufacturer_Part_Number (none) -> TMUX1204DQAR
- U2: Manufacturer_Name (none) -> Espressif Systems; Manufacturer_Part_Number (none) -> ESP32-S3-WROOM-1-N8R8
- U3: Manufacturer_Name (none) -> Analog Devices Inc./Maxim Integrated; Manufacturer_Part_Number (none) -> MAX98357AETE+T
- U4: Manufacturer_Name (none) -> Texas Instruments; Manufacturer_Part_Number (none) -> BQ25616RTWR
- U5: Manufacturer_Name (none) -> Nexperia USA Inc.; Manufacturer_Part_Number (none) -> PESD4USB5BTBS-QX
- U6: Manufacturer_Name (none) -> Texas Instruments; Manufacturer_Part_Number (none) -> TUSB321AIRWBR
