File: hardware/alarm_system_hardware/alarm_system_hardware.kicad_pcb (KiCad board)
At the start: 2 copper layers, 1 part, among them U1 ESP32-WROOM-32D

Commit message: Completed V0.01 PCB and production files
Parts:
- added BZ1: Buzzer, alarm_system:PS1440P02BT_TDK, F.Cu at (128.3, 68.8)
- added C1: 0.1uF, Capacitor_SMD:C_0805_2012Metric_Pad1.18x1.45mm_HandSolder, F.Cu at (137.0, 51.1)
- added C10: 1uF, Capacitor_SMD:C_0805_2012Metric_Pad1.18x1.45mm_HandSolder, F.Cu at (69.3, 79.4)
- added C11: 10uF, Capacitor_SMD:C_0805_2012Metric_Pad1.18x1.45mm_HandSolder, F.Cu at (79.5, 53.2)
- added C12: 10uF, Capacitor_SMD:C_0805_2012Metric_Pad1.18x1.45mm_HandSolder, F.Cu at (81.3, 82.0)
- added C13: 47nF, Capacitor_SMD:C_0805_2012Metric_Pad1.18x1.45mm_HandSolder, F.Cu at (77.9, 76.0)
- added C14: 4.7uF, Capacitor_SMD:C_0805_2012Metric_Pad1.18x1.45mm_HandSolder, F.Cu at (75.5, 75.9)
- added C15: 10uF, Capacitor_SMD:C_0805_2012Metric_Pad1.18x1.45mm_HandSolder, F.Cu at (72.4, 78.5)
- added C16: 0.1uF, Capacitor_SMD:C_0805_2012Metric_Pad1.18x1.45mm_HandSolder, F.Cu at (85.0, 61.3)
- added C17: 0.1uF, Capacitor_SMD:C_0805_2012Metric_Pad1.18x1.45mm_HandSolder, F.Cu at (65.1, 69.8)
- added C18: 0.1uF, Capacitor_SMD:C_0805_2012Metric_Pad1.18x1.45mm_HandSolder, F.Cu at (87.5, 38.4)
- added C19: 22uF, Capacitor_SMD:C_0805_2012Metric_Pad1.18x1.45mm_HandSolder, F.Cu at (84.4, 38.4)
- added C2: 1uF, Capacitor_SMD:C_0805_2012Metric_Pad1.18x1.45mm_HandSolder, F.Cu at (134.2, 51.0)
- added C20: 1uF, Capacitor_SMD:C_0805_2012Metric_Pad1.18x1.45mm_HandSolder, F.Cu at (78.5, 43.5)
- added C21: 22uF, Capacitor_SMD:C_0805_2012Metric_Pad1.18x1.45mm_HandSolder, F.Cu at (94.5, 75.7)
- added C22: 0.1uF, Capacitor_SMD:C_0805_2012Metric_Pad1.18x1.45mm_HandSolder, F.Cu at (110.7, 64.1)
- added C23: 1uF, Capacitor_SMD:C_0805_2012Metric_Pad1.18x1.45mm_HandSolder, F.Cu at (110.3, 84.8)
- added C24: 10uF, Capacitor_SMD:C_0805_2012Metric_Pad1.18x1.45mm_HandSolder, F.Cu at (81.3, 86.2)
- added C3: 1uF, Capacitor_SMD:C_0805_2012Metric_Pad1.18x1.45mm_HandSolder, F.Cu at (122.6, 84.9)
- added C4: 1uF, Capacitor_SMD:C_0805_2012Metric_Pad1.18x1.45mm_HandSolder, F.Cu at (148.3, 85.1)
- added C5: 1uF, Capacitor_SMD:C_0805_2012Metric_Pad1.18x1.45mm_HandSolder, F.Cu at (135.3, 84.9)
- added C6: 0.1uF, Capacitor_SMD:C_0805_2012Metric_Pad1.18x1.45mm_HandSolder, F.Cu at (144.9, 66.6)
- added C7: 10uF, Capacitor_SMD:C_0805_2012Metric_Pad1.18x1.45mm_HandSolder, F.Cu at (94.9, 69.0)
- added C8: 0.1uF, Capacitor_SMD:C_0805_2012Metric_Pad1.18x1.45mm_HandSolder, F.Cu at (87.3, 42.7)
- added C9: 10uF, Capacitor_SMD:C_0805_2012Metric_Pad1.18x1.45mm_HandSolder, F.Cu at (144.9, 69.0)
- added D1: GREEN LED, LED_SMD:LED_0805_2012Metric, F.Cu at (141.7, 86.5)
- added D10: RED LED, LED_SMD:LED_0805_2012Metric, F.Cu at (144.4, 86.5)
- added D11: LED, LED_SMD:LED_0805_2012Metric, F.Cu at (69.6, 85.2)
- added D12: RED LED, LED_SMD:LED_0805_2012Metric, F.Cu at (130.7, 86.5)
- added D13: RED LED, LED_SMD:LED_0805_2012Metric, F.Cu at (119.1, 86.5)
- added D15: LED, LED_SMD:LED_0805_2012Metric, F.Cu at (73.1, 90.6)
- added D2: GREEN LED, LED_SMD:LED_0805_2012Metric, F.Cu at (128.2, 86.5)
- added D3: GREEN LED, LED_SMD:LED_0805_2012Metric, F.Cu at (116.5, 86.5)
- added D4: LED, LED_SMD:LED_0805_2012Metric, F.Cu at (104.0, 76.8)
- added D5: LED, LED_SMD:LED_0805_2012Metric, F.Cu at (104.1, 79.3)
- added D6: LED, LED_SMD:LED_0805_2012Metric, F.Cu at (104.1, 81.9)
- added D7: LED, LED_SMD:LED_0805_2012Metric, F.Cu at (104.1, 84.7)
- added D8: LED, LED_SMD:LED_0805_2012Metric, F.Cu at (104.2, 87.4)
- added D9: TSD05DYFR, Diode_SMD:D_SOD-323_HandSoldering, F.Cu at (71.6, 52.8)
- added F1: Fuse, Fuse:Fuse_0805_2012Metric, F.Cu at (87.1, 85.0)
- added FB1: BBUP00321611121Y00, Resistor_SMD:R_1206_3216Metric_Pad1.30x1.75mm_HandSolder, F.Cu at (75.8, 54.0)
- added IC1: PCA9955BTW, alarm_system:SOP65P640X110-29N, F.Cu at (117.4, 68.3)
- added J1: Conn_02x04_Odd_Even, Connector_PinHeader_2.54mm:PinHeader_2x04_P2.54mm_Vertical, F.Cu at (135.6, 36.7)
- added J2: USB_C_Receptacle_USB2.0_16P, alarm_system:SAMESKY_UJ20-C-H-G-SMT-1-P16-TR, F.Cu at (61.1, 56.5)
- added J4: Conn_01x02_Socket, alarm_system:CONN_S2B-PH-K-S_JST, F.Cu at (151.2, 64.7)
- added J5: MSD-11-A, alarm_system:CUI_MSD-11-A, F.Cu at (148.6, 49.7)
- added J7: Conn_01x03_Socket, TerminalBlock_Phoenix:TerminalBlock_Phoenix_PT-1,5-3-3.5-H_1x03_P3.50mm_Horizontal, F.Cu at (87.4, 89.9)
- added L1: 1uH, alarm_system:IND_VLS5045EX-1R0N, F.Cu at (83.7, 77.3)
- added L2: 0.47uH, alarm_system:IND_IHLP-2020CZ-L, F.Cu at (100.8, 71.9)
- added Q1: AO3400A, Package_TO_SOT_SMD:SOT-23-3, F.Cu at (144.4, 76.0)
- added R1: 10k, Resistor_SMD:R_0805_2012Metric_Pad1.20x1.40mm_HandSolder, F.Cu at (132.9, 44.5)
- added R10: 330, Resistor_SMD:R_0805_2012Metric_Pad1.20x1.40mm_HandSolder, F.Cu at (78.4, 48.4)
- added R11: 47k, Resistor_SMD:R_0805_2012Metric_Pad1.20x1.40mm_HandSolder, F.Cu at (73.5, 48.5)
- added R12: 8.25k, Resistor_SMD:R_0805_2012Metric_Pad1.20x1.40mm_HandSolder, F.Cu at (110.2, 87.2)
- added R13: 330, Resistor_SMD:R_0805_2012Metric_Pad1.20x1.40mm_HandSolder, F.Cu at (110.2, 82.4)
- added R14: 100k, Resistor_SMD:R_0805_2012Metric_Pad1.20x1.40mm_HandSolder, F.Cu at (91.7, 85.0)
- added R15: 100k, Resistor_SMD:R_0805_2012Metric_Pad1.20x1.40mm_HandSolder, F.Cu at (96.2, 85.0)
- added R16: 0, Resistor_SMD:R_0805_2012Metric_Pad1.20x1.40mm_HandSolder, F.Cu at (95.5, 78.8)
- added R17: 0, Resistor_SMD:R_0805_2012Metric_Pad1.20x1.40mm_HandSolder, F.Cu at (105.7, 64.3)
- added R18: 10k, Resistor_SMD:R_0805_2012Metric_Pad1.20x1.40mm_HandSolder, F.Cu at (108.2, 66.4)
- added R19: 10k, Resistor_SMD:R_0805_2012Metric_Pad1.20x1.40mm_HandSolder, F.Cu at (106.8, 71.0)
- added R2: 10k, Resistor_SMD:R_0805_2012Metric_Pad1.20x1.40mm_HandSolder, F.Cu at (137.4, 42.2)
- added R20: 2k, Resistor_SMD:R_0805_2012Metric_Pad1.20x1.40mm_HandSolder, F.Cu at (110.0, 71.4)
- added R21: 4.7k, Resistor_SMD:R_0805_2012Metric_Pad1.20x1.40mm_HandSolder, F.Cu at (83.3, 48.7)
- added R22: 1k, Resistor_SMD:R_0805_2012Metric_Pad1.20x1.40mm_HandSolder, F.Cu at (141.0, 74.1)
- added R23: 4.7k, Resistor_SMD:R_0805_2012Metric_Pad1.20x1.40mm_HandSolder, F.Cu at (87.5, 48.8)
- added R24: 10k, Resistor_SMD:R_0805_2012Metric_Pad1.20x1.40mm_HandSolder, F.Cu at (82.1, 40.5)
- added R25: 909k, Resistor_SMD:R_0805_2012Metric_Pad1.20x1.40mm_HandSolder, F.Cu at (76.8, 64.4)
- added R26: 10k, Resistor_SMD:R_0805_2012Metric_Pad1.20x1.40mm_HandSolder, F.Cu at (82.5, 44.6)
- added R27: 200k, Resistor_SMD:R_0805_2012Metric_Pad1.20x1.40mm_HandSolder, F.Cu at (139.8, 66.9)
- added R28: 200k, Resistor_SMD:R_0805_2012Metric_Pad1.20x1.40mm_HandSolder, F.Cu at (139.8, 62.8)
- added R29: 100k, Resistor_SMD:R_0805_2012Metric_Pad1.20x1.40mm_HandSolder, F.Cu at (70.0, 82.7)
- added R3: 10k, Resistor_SMD:R_0805_2012Metric_Pad1.20x1.40mm_HandSolder, F.Cu at (137.4, 46.6)
- added R30: 10k, Resistor_SMD:R_0805_2012Metric_Pad1.20x1.40mm_HandSolder, F.Cu at (78.2, 87.3)
- added R31: 200, Resistor_SMD:R_0805_2012Metric_Pad1.20x1.40mm_HandSolder, F.Cu at (65.5, 85.1)
- added R32: 100k, Resistor_SMD:R_0805_2012Metric_Pad1.20x1.40mm_HandSolder, F.Cu at (71.5, 87.3)
- added R33: 200, Resistor_SMD:R_0805_2012Metric_Pad1.20x1.40mm_HandSolder, F.Cu at (72.2, 93.6)
- added R34: 10k, Resistor_SMD:R_0805_2012Metric_Pad1.20x1.40mm_HandSolder, F.Cu at (111.3, 53.2)
- added R35: 0, Resistor_SMD:R_0805_2012Metric_Pad1.20x1.40mm_HandSolder, F.Cu at (75.5, 93.3)
- added R36: 432, Resistor_SMD:R_0805_2012Metric_Pad1.20x1.40mm_HandSolder, F.Cu at (78.7, 92.2)
- added R37: 5.36k, Resistor_SMD:R_0805_2012Metric_Pad1.20x1.40mm_HandSolder, F.Cu at (81.4, 90.5)
- added R38: 31.6k, Resistor_SMD:R_0805_2012Metric_Pad1.20x1.40mm_HandSolder, F.Cu at (83.4, 92.6)
- added R39: 0, Resistor_SMD:R_0805_2012Metric_Pad1.20x1.40mm_HandSolder, F.Cu at (88.2, 70.0)
- added R4: 8.25k, Resistor_SMD:R_0805_2012Metric_Pad1.20x1.40mm_HandSolder, F.Cu at (122.5, 87.3)
- added R40: NC, Resistor_SMD:R_0805_2012Metric_Pad1.20x1.40mm_HandSolder, F.Cu at (90.5, 70.0)
- added R41: 511k, Resistor_SMD:R_0805_2012Metric_Pad1.20x1.40mm_HandSolder, F.Cu at (90.5, 78.2)
- added R42: 91k, Resistor_SMD:R_0805_2012Metric_Pad1.20x1.40mm_HandSolder, F.Cu at (90.5, 74.2)
- added R43: 0, Resistor_SMD:R_0805_2012Metric_Pad1.20x1.40mm_HandSolder, F.Cu at (78.8, 39.6)
- added R44: 1050, Resistor_SMD:R_0805_2012Metric_Pad1.20x1.40mm_HandSolder, F.Cu at (69.9, 75.0)
- added R45: 200, Resistor_SMD:R_0805_2012Metric_Pad1.20x1.40mm_HandSolder, F.Cu at (72.2, 67.5)
- added R46: 499, Resistor_SMD:R_0805_2012Metric_Pad1.20x1.40mm_HandSolder, F.Cu at (69.1, 66.4)
- added R47: 10M, Resistor_SMD:R_0805_2012Metric_Pad1.20x1.40mm_HandSolder, F.Cu at (71.3, 72.6)
- added R48: 10M, Resistor_SMD:R_0805_2012Metric_Pad1.20x1.40mm_HandSolder, F.Cu at (65.6, 73.1)
- added R49: 200k, Resistor_SMD:R_0805_2012Metric_Pad1.20x1.40mm_HandSolder, F.Cu at (79.0, 66.9)
- added R5: 8.25k, Resistor_SMD:R_0805_2012Metric_Pad1.20x1.40mm_HandSolder, F.Cu at (148.2, 87.4)
- added R50: 200k, Resistor_SMD:R_0805_2012Metric_Pad1.20x1.40mm_HandSolder, F.Cu at (83.2, 66.8)
- added R51: 0, Resistor_SMD:R_0805_2012Metric_Pad1.20x1.40mm_HandSolder, F.Cu at (144.9, 71.3)
- added R52: 0, Resistor_SMD:R_0805_2012Metric_Pad1.20x1.40mm_HandSolder, F.Cu at (129.9, 52.1)
- added R53: 330, Resistor_SMD:R_0805_2012Metric_Pad1.20x1.40mm_HandSolder, F.Cu at (141.2, 78.7)
- added R54: 100k, Resistor_SMD:R_0805_2012Metric_Pad1.20x1.40mm_HandSolder, F.Cu at (138.2, 77.8)
- added R6: 8.25k, Resistor_SMD:R_0805_2012Metric_Pad1.20x1.40mm_HandSolder, F.Cu at (135.2, 87.3)
- added R7: 330, Resistor_SMD:R_0805_2012Metric_Pad1.20x1.40mm_HandSolder, F.Cu at (122.6, 82.6)
- added R8: 330, Resistor_SMD:R_0805_2012Metric_Pad1.20x1.40mm_HandSolder, F.Cu at (148.2, 82.8)
- added R9: 330, Resistor_SMD:R_0805_2012Metric_Pad1.20x1.40mm_HandSolder, F.Cu at (135.2, 82.4)
- added REF**: MountingHole_3.2mm_M3, MountingHole:MountingHole_3.2mm_M3, F.Cu at (65.0, 92.7)
- added REF**: MountingHole_3.2mm_M3, MountingHole:MountingHole_3.2mm_M3, F.Cu at (154.0, 92.7)
- added REF**: MountingHole_3.2mm_M3, MountingHole:MountingHole_3.2mm_M3, F.Cu at (154.0, 33.0)
- added REF**: MountingHole_3.2mm_M3, MountingHole:MountingHole_3.2mm_M3, F.Cu at (65.0, 33.0)
- added SW1: SW_SPST, Button_Switch_SMD:SW_SPST_CK_RS282G05A3, F.Cu at (119.6, 92.6)
- added SW2: SW_SPST, Button_Switch_SMD:SW_SPST_CK_RS282G05A3, F.Cu at (144.4, 92.5)
- added SW3: SW_SPST, Button_Switch_SMD:SW_SPST_CK_RS282G05A3, F.Cu at (132.0, 92.5)
- added SW4: SW_Reed_Opener, TerminalBlock_Phoenix:TerminalBlock_Phoenix_PT-1,5-2-5.0-H_1x02_P5.00mm_Horizontal, F.Cu at (66.7, 40.1)
- added SW5: SW_SPST, Button_Switch_SMD:SW_SPST_CK_RS282G05A3, F.Cu at (107.1, 92.6)
- added SW7: SW_Tactile, Button_Switch_SMD:SW_SPST_CK_RS282G05A3, F.Cu at (74.5, 41.5)
- added SW8: SW_Tactile, Button_Switch_SMD:SW_SPST_CK_RS282G05A3, F.Cu at (118.5, 54.1)
- added TP1: TestPoint, TestPoint:TestPoint_Pad_D1.0mm, F.Cu at (84.8, 56.3)
- added TP10: TestPoint, TestPoint:TestPoint_Pad_D1.0mm, F.Cu at (85.9, 59.2)
- added TP2: TestPoint, TestPoint:TestPoint_Pad_D1.0mm, F.Cu at (82.7, 58.5)
- added TP3: TestPoint, TestPoint:TestPoint_Pad_D1.0mm, F.Cu at (78.8, 60.6)
- added TP4: TestPoint, TestPoint:TestPoint_Pad_D1.0mm, F.Cu at (75.5, 68.5)
- added TP5: TestPoint, TestPoint:TestPoint_Pad_D1.0mm, F.Cu at (76.0, 72.0)
- added TP6: TestPoint, TestPoint:TestPoint_Pad_D1.0mm, F.Cu at (67.0, 75.8)
- added TP7: TestPoint, TestPoint:TestPoint_Pad_D1.0mm, F.Cu at (74.0, 63.1)
- added TP8: TestPoint, TestPoint:TestPoint_Pad_D1.0mm, F.Cu at (86.7, 65.2)
- added TP9: TestPoint, TestPoint:TestPoint_Pad_D1.0mm, F.Cu at (76.4, 60.6)
- added U10: TMUX1204DQAR, alarm_system:USON10_DQA_TEX, F.Cu at (68.1, 70.1)
- added U2: ESP32-S3-WROOM-1-N8R8, RF_Module:ESP32-S3-WROOM-1, F.Cu at (99.5, 42.9)
- added U3: MAX98357A, Package_DFN_QFN:TQFN-16-1EP_3x3mm_P0.5mm_EP1.23x1.23mm, F.Cu at (145.5, 63.0)
- added U4: BQ25616JRTWR, alarm_system:WQFN24_RTW_TEX, F.Cu at (75.8, 82.5)
- added U5: PESD4USB5BTBS-QX, Package_DFN_QFN:Diodes_UDFN-10_1.0x2.5mm_P0.5mm, F.Cu at (72.7, 57.8)
- added U6: TUSB321AIRWBR, Package_DFN_QFN:Texas_X2QFN-12_1.6x1.6mm_P0.4mm, F.Cu at (81.0, 62.7)
- U1: value ESP32-WROOM-32D -> TPS63802DLAR; footprint RF_Module:ESP32-WROOM-32D -> alarm_system:DLA0010A
- moved U1 52.9 mm to (94.7, 72.1)
Connections:
- U1 pad 1: Net-(U1-GND-Pad1) -> CHARGER_POWER
- U1 pad 10: unconnected-(U1-IO25-Pad10) -> CHARGER_POWER
- U1 pad 2: unconnected-(U1-VDD-Pad2) -> Net-(U1-MODE)
- U1 pad 3: unconnected-(U1-EN-Pad3) -> GND
- U1 pad 4: unconnected-(U1-SENSOR_VP-Pad4) -> Net-(U1-FB)
- U1 pad 6: unconnected-(U1-IO34-Pad6) -> Net-(U1-VOUT)
- U1 pad 7: unconnected-(U1-IO35-Pad7) -> Net-(U1-L2)
- U1 pad 8: unconnected-(U1-IO32-Pad8) -> GND
- U1 pad 9: unconnected-(U1-IO33-Pad9) -> Net-(U1-L1)
Routing:
- net GND: track 0.00 -> 160.3 mm, vias 0 -> 130
- net UBSC_VBUS: track 0.00 -> 77.8 mm, vias 0 -> 2
- net ARM_SWITCH: track 0.00 -> 68.6 mm, vias 0 -> 2
- net BUZZER_GPIO: track 0.00 -> 66.6 mm, vias 0 -> 2
- net AUDIO_ON_OFF_SWITCH: track 0.00 -> 57.0 mm, vias 0 -> 2
- net SDCARD_WP: track 0.00 -> 55.8 mm, vias 0 -> 2
- net SDCARD_CD: track 0.00 -> 55.4 mm, vias 0 -> 2
- net SDCARD_CD/CS: track 0.00 -> 54.2 mm, vias 0 -> 2
- net +3V3: track 0.00 -> 51.9 mm, vias 0 -> 40
- net SDA: track 0.00 -> 48.6 mm, vias 0 -> 2
- net DAC_GAIN_DRV: track 0.00 -> 47.2 mm, vias 0 -> 2
- net DAC_!SD_BOOT: track 0.00 -> 46.3 mm, vias 0 -> 2
- net NOTIFICATIONS_SWITCH: track 0.00 -> 45.8 mm, vias 0 -> 2
- net SCL: track 0.00 -> 45.3 mm, vias 0 -> 2
- net ESP_DIN: track 0.00 -> 45.2 mm
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- added copper zone on In2.Cu, net +3V3
- added copper zone on F.Cu, net GND
- added copper zone on In1.Cu, net GND
- added copper zone on F.Cu, net Net-(C13-Pad2)
Other:
- board outline added: 97 x 67.7 mm
- copper layers 2 -> 4
- board text added: "3V3"
- board text added: "Arm"
- board text added: "Audio"
- board text added: "BOOT"
- board text added: "Battery"
- board text added: "Battery Life"
- board text added: "GND"
- board text added: "MTCK"
- board text added: "MTDI"
- board text added: "MTDO"
- board text added: "MTMS"
- board text added: "Notifications"
- board text added: "RESET"
- board text added: "RX0"
- board text added: "Reed"
- board text added: "Speaker"
- board text added: "TS"
- board text added: "TX0"
- board text added: "V+"
- board text added: "V-"
- board text added: "speaker size"

Commit message: PCBA export file and related hardware changes
Parts:
- D11, D15, D4, D5, D6, D7, D8: value LED -> GREEN LED
- IC1: value PCA9955BTW -> PCA9955BTWJ
- J7: footprint TerminalBlock_Phoenix:TerminalBlock_Phoenix_PT-1,5-3-3.5-H_1x03_P3.50mm_Horizontal -> TerminalBlock_Phoenix:TerminalBlock_Phoenix_PT-1,5-3-5.0-H_1x03_P5.00mm_Horizontal
- R27, R28: value 200k -> 100k
- SW7, SW8: value SW_Tactile -> SW_SPST
- moved R14 1.81 mm to (93.1, 83.9)
- moved R15 1.62 mm to (97.4, 83.8)
- moved F1 1.19 mm to (87.1, 83.8)
- moved J7 0.30 mm to (87.4, 89.7)
- moved R37 0.24 mm to (81.1, 90.5)
- moved R38 0.19 mm to (83.2, 92.6)
Connections:
- J2 pad A4_B9: /USBC_VBUS -> (no net)
- J2 pad B4_A9: /USBC_VBUS -> (no net)
Routing:
- net V_BAT: track 7.82 -> 9.85 mm
- net BAT_REGN: track 19.8 -> 18.8 mm
- net V_BAT_ADC: track 38.4 -> 39.0 mm
